File: ESP32_board/ESP-32_USB_sequencer/ESP-32_USB_sequencer.kicad_pcb (KiCad board)
At the start: 2 copper layers, 31 parts, among them J1 AudioJack2_SwitchT, J3 AudioJack3, J5 AudioJack2_SwitchT, J6 AudioJack2_SwitchT, J7 AudioJack2_SwitchT, Q2 Q_NMOS_GSD, U1 mini_esp32, U3 MCP4728, U4 TL074

Commit message: lots of stuff
Parts:
- removed D10: D_Schottky, Diode_THT:D_5W_P12.70mm_Horizontal
- removed I2CB1: Conn_01x04_Pin, Connector_PinHeader_2.54mm:PinHeader_1x04_P2.54mm_Vertical
- added C1: C_Small, Capacitor_SMD:C_0805_2012Metric_Pad1.18x1.45mm_HandSolder, F.Cu at (104.4, 171.6)
- added C2: C_Polarized_US, Capacitor_THT:CP_Radial_D8.0mm_P5.00mm, F.Cu at (132.2, 92.7)
- added C3: C_Small, Capacitor_SMD:C_0805_2012Metric_Pad1.18x1.45mm_HandSolder, F.Cu at (87.6, 165.5)
- added I2CA2: Conn_01x04_Socket, Connector_PinHeader_2.54mm:PinHeader_1x04_P2.54mm_Vertical, B.Cu at (135.9, 114.1)
- added J10: MIDI_in, Connector_Audio:Jack_3.5mm_QingPu_WQP-PJ398SM_Vertical_CircularHoles_1, B.Cu at (120.7, 158.8)
- added J12: MIDI_out, Connector_Audio:Jack_3.5mm_QingPu_WQP-PJ398SM_Vertical_CircularHoles_1, B.Cu at (136.6, 158.8)
- added J2: AudioJack2_SwitchT, Connector_Audio:Jack_3.5mm_QingPu_WQP-PJ398SM_Vertical_CircularHoles, B.Cu at (100.3, 158.8)
- added Q1: BSS138, Package_TO_SOT_SMD:SOT-23, F.Cu at (135.0, 139.5)
- added Q3: 2n2222, Package_TO_SOT_THT:TO-92_Inline_Wide, F.Cu at (91.4, 141.1)
- added Q4: 2n2222, Package_TO_SOT_THT:TO-92_Inline_Wide, F.Cu at (81.3, 140.8)
- added Q7: 2n2222, Package_TO_SOT_THT:TO-92_Inline_Wide, F.Cu at (118.1, 143.3)
- added R10: 10k, Resistor_THT:R_Axial_DIN0207_L6.3mm_D2.5mm_P10.16mm_Horizontal, F.Cu at (127.0, 129.3)
- added R11: 10k, Resistor_THT:R_Axial_DIN0207_L6.3mm_D2.5mm_P10.16mm_Horizontal, F.Cu at (127.0, 134.4)
- added R12: 10k, Resistor_THT:R_Axial_DIN0207_L6.3mm_D2.5mm_P10.16mm_Horizontal, F.Cu at (127.0, 145.8)
- added R13: 10k, Resistor_THT:R_Axial_DIN0207_L6.3mm_D2.5mm_P10.16mm_Horizontal, F.Cu at (127.0, 150.9)
- added R14: 1M, Resistor_THT:R_Axial_DIN0207_L6.3mm_D2.5mm_P10.16mm_Horizontal, F.Cu at (99.1, 147.5)
- added R15: 100k, Resistor_THT:R_Axial_DIN0207_L6.3mm_D2.5mm_P10.16mm_Horizontal, F.Cu at (85.1, 152.2)
- added R16: 1M, Resistor_THT:R_Axial_DIN0207_L6.3mm_D2.5mm_P10.16mm_Horizontal, F.Cu at (85.1, 147.1)
- added R17: 4.7k, Resistor_SMD:R_0805_2012Metric_Pad1.20x1.40mm_HandSolder, F.Cu at (82.5, 165.1)
- added R18: 100k, Resistor_THT:R_Axial_DIN0207_L6.3mm_D2.5mm_P10.16mm_Horizontal, F.Cu at (81.3, 129.5)
- added R19: 100k, Resistor_THT:R_Axial_DIN0207_L6.3mm_D2.5mm_P10.16mm_Horizontal, F.Cu at (81.3, 134.6)
- added R21: 4.7k, Resistor_THT:R_Axial_DIN0207_L6.3mm_D2.5mm_P10.16mm_Horizontal, F.Cu at (111.8, 129.3)
- added R22: 220R, Resistor_THT:R_Axial_DIN0207_L6.3mm_D2.5mm_P10.16mm_Horizontal, F.Cu at (106.7, 129.3)
- added R23: 220R, Resistor_THT:R_Axial_DIN0207_L6.3mm_D2.5mm_P10.16mm_Horizontal, F.Cu at (101.6, 152.2)
- added R24: 100k, Resistor_THT:R_Axial_DIN0207_L6.3mm_D2.5mm_P10.16mm_Horizontal, F.Cu at (124.5, 135.7)
- added R27: 220R, Resistor_THT:R_Axial_DIN0207_L6.3mm_D2.5mm_P10.16mm_Horizontal, F.Cu at (114.3, 149.6)
- added U5: 6N138, Package_DIP:DIP-8_W7.62mm, F.Cu at (102.9, 148.4)
- D1, D2, D3, D4, D5, D6, D7, D8: footprint Diode_THT:D_5W_P12.70mm_Horizontal -> Diode_SMD:D_SOD-123
- D9: value D_Schottky -> 1n914
- I2CA1, J1, J5, J6, J7: moved to B.Cu
- J3: value AudioJack3 -> AudioJack2_SwitchT; footprint ih_kicad:PJ-392-vertical-TRS-3.5mm -> Connector_Audio:Jack_3.5mm_QingPu_WQP-PJ398SM_Vertical_CircularHoles; moved to B.Cu
- Q2: value Q_NMOS_GSD -> BSS138
- R1, R2, R3, R4: value R_Small_US -> 100R; footprint Resistor_THT:R_Axial_DIN0207_L6.3mm_D2.5mm_P10.16mm_Horizontal -> Resistor_SMD:R_0805_2012Metric_Pad1.20x1.40mm_HandSolder
- R5: value R_Small_US -> 100k
- R6, R7, R8, R9: value R_Small_US -> 10k; footprint Resistor_THT:R_Axial_DIN0207_L6.3mm_D2.5mm_P10.16mm_Horizontal -> Resistor_SMD:R_0805_2012Metric_Pad1.20x1.40mm_HandSolder
- U4: footprint Package_DIP:DIP-14_W7.62mm -> Package_SO:SOIC-14_3.9x8.7mm_P1.27mm
- moved D2 205.4 mm to (83.0, 172.8)
- moved J6 201.8 mm to (84.5, 181.6), turned to 90 degrees
- moved R2 200.5 mm to (105.6, 176.6)
- moved D3 200.4 mm to (115.7, 176.8), turned to 180 degrees
- moved J1 198.1 mm to (117.4, 181.6), turned to 90 degrees
- moved D4 194.0 mm to (115.7, 172.8), turned to 180 degrees
- moved D1 186.5 mm to (83.0, 176.6), turned to 180 degrees
- moved R1 178.6 mm to (76.2, 172.7)
- moved J3 164.6 mm to (84.5, 158.8), turned to 90 degrees
- moved R6 163.1 mm to (77.9, 176.6), turned to 180 degrees
- moved R4 153.6 mm to (89.7, 176.6)
- moved J7 150.0 mm to (101.0, 181.6), turned to 90 degrees
- moved U3 148.3 mm to (92.7, 165.5)
- moved R9 144.3 mm to (94.8, 176.6), turned to 180 degrees
- moved R5 139.1 mm to (99.1, 152.5), turned to 180 degrees
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Connections:
- net Net-(U3-VOUTA) renamed /DAC_A
- net Net-(U3-VOUTD) renamed /DAC_D
- D9 pad 1: Net-(D10-A) -> Net-(D9-K)
- D9 pad 2: GND -> Net-(D9-A)
- I2CA1 pad 1: unconnected-(I2CA1-Pin_1-Pad1) -> /5v_SCL
- I2CA1 pad 2: unconnected-(I2CA1-Pin_2-Pad2) -> /5v_SDA
- I2CA1 pad 3: unconnected-(I2CA1-Pin_3-Pad3) -> +5V
- I2CA1 pad 4: unconnected-(I2CA1-Pin_4-Pad4) -> GND
- J1 pad TN: unconnected-(J1-PadTN) -> GND
- J3 pad S: Net-(J3-PadS) -> GND
- J3 pad T: unconnected-(J3-PadT) -> Net-(J3-PadT)
- J5 pad TN: unconnected-(J5-PadTN) -> GND
- J6 pad TN: unconnected-(J6-PadTN) -> GND
- J7 pad TN: unconnected-(J7-PadTN) -> GND
- Q2 pad 1: unconnected-(Q2-G-Pad1) -> +3.3V
- Q2 pad 2: unconnected-(Q2-S-Pad2) -> /SDA
- Q2 pad 3: unconnected-(Q2-D-Pad3) -> /5v_SDA
- R5 pad 1: Net-(J3-PadS) -> Net-(J2-PadT)
- R5 pad 2: Net-(D10-A) -> Net-(Q3-B)
- U1 pad 24: unconnected-(U1-IO_27-Pad24) -> /GPIO27
- U1 pad 26: unconnected-(U1-IO_25-Pad26) -> /INT
- U1 pad 29: /INT -> /midi_out
- U1 pad 31: unconnected-(U1-IO_16/D4-Pad31) -> /midi_in
- U3 pad 4: unconnected-(U3-~{LDAC}-Pad4) -> Net-(U3-~{LDAC})
- U3 pad 7: Net-(U3-VOUTB) -> /DAC_B
- U3 pad 8: Net-(U3-VOUTC) -> /DAC_C
- U4 pad 10: Net-(U3-VOUTB) -> /DAC_C
- U4 pad 11: unconnected-(U4E-V--Pad11) -> GND
- U4 pad 4: unconnected-(U4E-V+-Pad4) -> +5V
- U4 pad 5: Net-(U3-VOUTC) -> /DAC_B
Routing:
- net +5V: track 0.00 -> 337.7 mm, vias 0 -> 6
- net GND: track 0.00 -> 213.8 mm, vias 0 -> 5
- net +3.3V: track 0.00 -> 212.4 mm
- net /5v_SCL: track 0.00 -> 136.2 mm
- net /5v_SDA: track 0.00 -> 131.3 mm, vias 0 -> 4
- net /SCL: track 0.00 -> 66.3 mm
- net /A32: track 0.00 -> 60.4 mm
- net /midi_in: track 0.00 -> 59.9 mm, vias 0 -> 1
- net /GPIO27: track 0.00 -> 59.3 mm
- net /SDA: track 0.00 -> 52.0 mm
- net /MISO: track 0.00 -> 49.2 mm
- net /CS: track 0.00 -> 49.2 mm
- net /MOSI: track 0.00 -> 49.2 mm
- net /CLK: track 0.00 -> 49.2 mm
- net /midi_out: track 0.00 -> 48.0 mm, vias 0 -> 1
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- added copper zone on B.Cu, net GND
Other:
- board outline added: 69.8 x 102.9 mm
- board text added: "3v"
- board text added: "5v"
- board text added: "5v SCL"
- board text added: "5v SDA"
- board text added: "Clock"
- board text added: "GND"
- board text added: "MIDI IN"
- board text added: "MIDI OUT"
- board text added: "Reset"
