File: ESP32_board/ESP-32_USB_sequencer/ESP-32_USB_sequencer.kicad_sch (KiCad schematic)
At the start: 37 parts, among them J1 AudioJack2_SwitchT, J3 AudioJack3, J5 AudioJack2_SwitchT, J6 AudioJack2_SwitchT, J7 AudioJack2_SwitchT, Q1 BSS138, Q2 BSS138, U1 mini_esp32, U3 MCP4728, U4 TL074, U5 TL074

Commit message: lots of stuff
Parts:
- removed D10: D_Schottky, Diode_THT:D_5W_P12.70mm_Horizontal, symbol Device:D_Schottky
- removed I2CB1: Conn_01x04_Pin, Connector_PinHeader_2.54mm:PinHeader_1x04_P2.54mm_Vertical, symbol Connector:Conn_01x04_Pin
- removed J3: AudioJack3, ih_kicad:PJ-392-vertical-TRS-3.5mm, symbol Connector_Audio:AudioJack3
- removed U5: TL074, symbol Amplifier_Operational:TL074
- added C1, C3: C_Small, Capacitor_SMD:C_0805_2012Metric_Pad1.18x1.45mm_HandSolder, symbol Device:C_Small
- added C2: C_Polarized_US, Capacitor_THT:CP_Radial_D8.0mm_P5.00mm, symbol Device:C_Polarized_US
- added I2CA2: Conn_01x04_Socket, Connector_PinHeader_2.54mm:PinHeader_1x04_P2.54mm_Vertical, symbol Connector:Conn_01x04_Socket
- added J10: MIDI_in, Connector_Audio:Jack_3.5mm_QingPu_WQP-PJ398SM_Vertical_CircularHoles_1, symbol Connector_Audio:AudioJack3
- added J12: MIDI_out, Connector_Audio:Jack_3.5mm_QingPu_WQP-PJ398SM_Vertical_CircularHoles_1, symbol Connector_Audio:AudioJack3
- added J2, J3: AudioJack2_SwitchT, Connector_Audio:Jack_3.5mm_QingPu_WQP-PJ398SM_Vertical_CircularHoles, symbol Connector_Audio:AudioJack2_SwitchT
- added Q3, Q4, Q7: 2n2222, Package_TO_SOT_THT:TO-92_Inline_Wide, symbol Simulation_SPICE:NPN
- added R14, R16: 1M, Resistor_THT:R_Axial_DIN0207_L6.3mm_D2.5mm_P10.16mm_Horizontal, symbol Device:R_Small_US
- added R15, R18, R19, R24: 100k, Resistor_THT:R_Axial_DIN0207_L6.3mm_D2.5mm_P10.16mm_Horizontal, symbol Device:R_Small_US
- added R17: 4.7k, Resistor_SMD:R_0805_2012Metric_Pad1.20x1.40mm_HandSolder, symbol Device:R_Small_US
- added R21: 4.7k, Resistor_THT:R_Axial_DIN0207_L6.3mm_D2.5mm_P10.16mm_Horizontal, symbol Device:R_Small_US
- added R22, R23, R27: 220R, Resistor_THT:R_Axial_DIN0207_L6.3mm_D2.5mm_P10.16mm_Horizontal, symbol Device:R_Small_US
- added U5: 6N138, Package_DIP:DIP-8_W7.62mm, symbol Isolator:6N138
- D1, D2, D3, D4, D5, D6, D7, D8: footprint Diode_THT:D_5W_P12.70mm_Horizontal -> Diode_SMD:D_SOD-123
- D9: value D_Schottky -> 1n914
- R1, R2, R3, R4: value R_Small_US -> 100R; footprint Resistor_THT:R_Axial_DIN0207_L6.3mm_D2.5mm_P10.16mm_Horizontal -> Resistor_SMD:R_0805_2012Metric_Pad1.20x1.40mm_HandSolder
- R5: value R_Small_US -> 100k
- R6, R7, R8, R9: value R_Small_US -> 10k; footprint Resistor_THT:R_Axial_DIN0207_L6.3mm_D2.5mm_P10.16mm_Horizontal -> Resistor_SMD:R_0805_2012Metric_Pad1.20x1.40mm_HandSolder
- U4: footprint Package_DIP:DIP-14_W7.62mm -> Package_SO:SOIC-14_3.9x8.7mm_P1.27mm
Connections:
- net +3.3V: now also R18.2, R19.2, R22.2, U5.8 (VCC)
- net +5V: now also I2CA1.3 (Pin_3), U4.4 (V+), C1.2, C2.1, C3.2, I2CA2.3 (Pin_3), R27.1
- net 5v_SCL: now also I2CA1.1 (Pin_1), I2CA2.1 (Pin_1)
- net 5v_SDA: now also I2CA1.2 (Pin_2), I2CA2.2 (Pin_2)
- net A32: now also Q4.1 (C), R18.1
- net GND: now also I2CA1.4 (Pin_4), J1.TN, J5.TN, J6.TN, J7.TN, U4.11 (V-), C1.1, C2.2, C3.1, I2CA2.4 (Pin_4), J10.S, J12.S, J2.S, J2.TN, J3.S, J3.TN, Q3.3 (E), Q4.3 (E), Q7.3 (E), R14.1, R16.1, R17.1, R21.1, U5.5 (GND); no longer D9.2 (A)
- net INT: now also U1.26 (IO_25); no longer U1.29 (IO_17/D3)
- net at R5.2: now also Q3.2 (B), R14.2; no longer D9.1 (K)
- net DAC_D: now reaches U3.9 (VOUTD), U4.12 (+)
- net DAC_B: now reaches U4.5 (+)
- net DAC_B: now also U3.7 (VOUTB); no longer U3.8 (VOUTC)
- net at U3.4 (~{LDAC}): now also R17.2
- net DAC_A: now reaches U3.6 (VOUTA), U4.3 (+)
- net DAC_C: now reaches U4.10 (+)
- net DAC_C: now also U3.8 (VOUTC); no longer U3.7 (VOUTB)
- net GPIO27: now reaches U1.24 (IO_27)
- net GPIO27: now also Q3.1 (C), R19.1
- net midi_in: now reaches U1.31 (IO_16/D4)
- net midi_in: now also R22.1, U5.6 (VO2)
- net at R5.1: now also J2.T
- new net: J10.R, R23.2
- new net: D9.2 (A), J10.T, U5.3 (C2)
- new net: R21.2, U5.7 (VO1)
- new net: Q4.2 (B), R15.2, R16.2
- new net: D9.1 (K), R23.1, U5.2 (C1)
- new net: J12.R, R27.2
- new net: J3.T, R15.1
- new net: J12.T, Q7.1 (C)
- new net: Q7.2 (B), R24.2
- new net midi_out: R24.1, U1.29 (IO_17/D3)
Other:
- note added: "A-6115 Stereo 3.5mm jack"
- moved on the sheet: R5, U2
