File: ESP32_board/Grand_central_pcb_simple/Grand_central_pcb_simple.kicad_sch (KiCad schematic)
At the start: 49 parts, among them J1 MIDI_out, J2 DAC, J3 DAC1, J4 CLK, SW1 RotaryEncoder_Switch, SW3 SW_Push, U1 mini_esp32, U2 TL074

Commit message: grand
Other:
- note added: "Inverted comparator circuit- for both reset and midi output midi needs to be not inverted!!!"
- note added: "move led to opamp output"
- note removed: "Inverted comparator circuit- for both reset and midi output"
